File: KiCAD/udb-cy.kicad_pcb (KiCad board)
At the start: 4 copper layers, 18 x 16.5 mm, 15 parts, among them J1 SM04B-SRSS-TB(LF)(SN), J2 USB_C_Receptacle

Commit message: Added JST SUR connector option
Parts:
- added J2: JST_SUR_4, Connector_JST:JST_SUR_SM04B-SURS-TF_1x04-1MP_P0.80mm_Horizontal, F.Cu at (103.0, 53.0)
- renumbered J2 to J0
Routing:
- net VCC: track 14.4 -> 17.6 mm
- net D-: track 13.0 -> 15.3 mm
- net D+: track 14.0 -> 15.3 mm
- net GND: track 13.1 -> 14.3 mm, vias 13 -> 15
Other:
- board text added: "Y"

Commit message: Expose all 4 pins on the underside
Parts:
- removed TP-Gnd1, TP-Vcc1: TestPoint, TestPoint:TestPoint_Pad_1.5x1.5mm
- added J3: Conn_01x04, PCM_SparkFun-Connector:1x04_P2.54mm_SolderPads, B.Cu at (103.1, 53.2)
- H1: value MountingHole_Pad -> ~; footprint MountingHole:MountingHole_2.2mm_M2_Pad -> ts-kicad-lib:Mount_M2_Rel
- H2, H3, H4: value MountingHole -> ~; footprint MountingHole:MountingHole_2.2mm_M2 -> ts-kicad-lib:Hole_M2
- J1: value SM04B-SRSS-TB(LF)(SN) -> JST-SH-04
- J2: value JST_SUR_4 -> JST-SUR-04
Routing:
- net D-: track 15.3 -> 20.7 mm, vias 2 -> 3
- net VBUS: track 18.4 -> 22.1 mm, vias 4 -> 3
- net D+: track 15.3 -> 17.7 mm
- net GND: track 14.3 -> 12.5 mm, vias 15 -> 11
- net Net-(J0-CC2): track 10.1 -> 9.38 mm
- net VCC: track 17.6 -> 16.9 mm
- net Earth: vias 4 -> 6
Other:
- board text added: "+"
- board text added: "+5V"
- board text added: "-"
- board text removed: "Vcc"
- board text removed: "Y"

Commit message: .
Parts:
- added C2: 1nF, Capacitor_SMD:C_0603_1608Metric, F.Cu at (110.8, 48.3)
- added FB1: 600Ω @ 100MHz, Inductor_SMD:L_0603_1608Metric, F.Cu at (109.3, 44.6)
- C1: value 4.7uF -> 0.1µF
- moved C1 3.70 mm to (109.3, 48.3), turned to 90 degrees
- moved R2 2.28 mm to (106.1, 48.3), turned to 90 degrees
- moved R1 0.80 mm to (107.6, 48.3), turned to 90 degrees
- moved R3 0.08 mm to (110.8, 44.6)
Routing:
- net GND: track 12.0 -> 23.0 mm, vias 11 -> 9
- net Earth: track 3.91 -> 13.6 mm, vias 6 -> 8
- net Net-(J0-CC1): track 6.24 -> 9.08 mm

Commit message: updated
Parts:
- J1: footprint Connector_JST:JST_SH_SM04B-SRSS-TB_1x04-1MP_P1.00mm_Horizontal -> ts-keyboard-lib:JST_SH_SM04B-SRSS-TB_1x04-1MP_P1.00mm_Horizontal
- R1, R2, R3: footprint Resistor_SMD:R_0603_1608Metric -> Resistor_SMD:R_0603_1608Metric_Pad0.98x0.95mm_HandSolder
Connections:
- J0 pad SH: (no net) -> Earth
Routing:
- net VBUS: track 21.8 -> 14.4 mm, vias 3 -> 0
- net Earth: track 13.6 -> 15.0 mm
- net D-: track 20.4 -> 19.9 mm
